File: hackspace cube/hackspace cube/Cube pcb/Cube pcb - with ground plain.kicad_pcb (KiCad board)
At the start: 2 copper layers, 100 x 64.5 mm, 61 parts, among them J1 Conn_01x09 ( conector 1), J2 Conn_01x09 ( conector 2), J3 Conn_01x02 ( exstra ground co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, J4 Conn_01x14 ( Spare Ports ), Q1 BSS138, Q10 BSS138, Q11 BSS138, Q12 BSS138, Q13 BSS138, Q14 BSS138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

Commit message: ground plain added
ground plain added
Routing:
- added copper zone on B.Cu, net GND
- added copper zone on F.Cu, net GND
Changed lines of the file:
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@@
 		)
 	)
+	(gr_text "GND"
+		(at 86.5 94.5 0)
+		(layer "F.SilkS")
+		(effects
+			(font
+				(size 1 1)
+				(thickness 0.1)
+			)
+			(justify left bottom)
+		)
+	)
 	(gr_text "GIPO7"
 		(at 109 86 0)
@@
 		)
 	)
+	(gr_text "GND"
+		(at 86 120 0)
+		(layer "F.SilkS")
+		(effects
+			(font
+				(size 1 1)
+				(thickness 0.1)
+			)
+			(justify left bottom)
+		)
+	)
 	(gr_text "D-1"
 		(at 109.5 83 0)
@@
 		)
 	)
-	(gr_text "GND"
-		(at 86.5 94.58 0)
-		(layer "Edge.Cuts")
-		(effects
-			(font
-				(size 1 1)
-				(thickness 0.15)
-			)
-			(justify left bottom)
-		)
-	)
 	(gr_text "one"
 		(at 186.5 183.5 0)
@@
 		)
 	)
-	(gr_text "GND"
-		(at 86 120.08 0)
-		(layer "Edge.Cuts")
-		(effects
-			(font
-				(size 1 1)
-				(thickness 0.15)
-			)
-			(justify left bottom)
-		)
-	)
 	(gr_text "1.3"
 		(at 269 193.5 0)
@@
 		(net 49)
 	)
+	(zone
+		(net 6)
+		(net_name "GND")
+		(layers "F.Cu" "B.Cu")
+		(hatch edge 0.5)
+		(connect_pads
+			(clearance 0.5)
+		)
+		(min_thickness 0.25)
+		(filled_areas_thickness no)
+		(fill yes
+			(thermal_gap 0.5)
+			(thermal_bridge_width 0.5)
+		)
+		(polygon
+			(pts
+				(xy 175 65) (xy 75 65) (xy 75 129.5) (xy 175 129.5)
+			)
+		)
+	)
 	(group ""
