File: hackspace cube/hackspace cube/Cube pcb/Cube pcb - with ground plain2.kicad_pcb (KiCad board)
At the start: 2 copper layers, 100 x 64.5 mm, 67 parts, among them J1 Conn_01x09 ( conector 1), J2 Conn_01x09 ( conector 2), J3 Conn_01x02 ( exstra ground co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, J4 Conn_01x14 ( Spare Ports ), Q1 BSS138, Q10 BSS138, Q11 BSS138, Q12 BSS138, Q13 BSS138, Q14 BSS138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

Commit message: updated spelling
updated spelling using NavSpellCheck
Other:
- board text added: "GPIO0"
- board text added: "GPIO1"
- board text added: "GPIO10"
- board text added: "GPIO11"
- board text added: "GPIO12"
- board text added: "GPIO13"
- board text added: "GPIO14"
- board text added: "GPIO15"
- board text added: "GPIO2"
- board text added: "GPIO3"
- board text added: "GPIO4"
- board text added: "GPIO5"
- board text added: "GPIO6"
- board text added: "GPIO7"
- board text added: "GPIO8"
- board text added: "GPIO9"
- board text added: "PCB DESIGNED BY SAMSON B LEEDS HACKSPACE CUBE CONTROL BOARD CAN BE FOUND ON GITHUB AT www.github.com/bozzer91 IF NOT ON LEEDS HACKSPACE GITHUB LICENCE: OPEN SOURCE"
- board text added: "REF FOR BOARD D- = DATA THEN LINE OUPUT NUMBER 1 = A NUMBER BY ITS LEFT NEXT TO THE PICO LABLES THE GPIO NUMBER OF THAT PIN TEST POINTS GPIO = RIGHT OF RESISTOR D- = LEFT OF THE RESISTOR"
- board text removed: "GIPO0"
- board text removed: "GIPO1"
- board text removed: "GIPO10"
- board text removed: "GIPO11"
- board text removed: "GIPO12"
- board text removed: "GIPO13"
- board text removed: "GIPO14"
- board text removed: "GIPO15"
- board text removed: "GIPO2"
- board text removed: "GIPO3"
- board text removed: "GIPO4"
- board text removed: "GIPO5"
- board text removed: "GIPO6"
- board text removed: "GIPO7"
- board text removed: "GIPO8"
- board text removed: "GIPO9"
- board text removed: "PCB DESIGNED BY SAMSON B LEEDS HACKSPACE CUBE CONTROLL BAORD CAN BE FOUND ON GITHUB AT www.github.com/bozzer91 IF NOT ON LEEDS HACKSPACE GITHUB LICENCE: OPEN SOURCE"
- board text removed: "REFF FOR BAORD D- = DATA THEN LINE OUPUT NUMBER 1 = A NUMBER BY ITS LEFT NEXT TO THE PICO LABLES THE GPIO NUMBER OF THAT PIN TEST POINTS GPIO = RIGHT OF RESISTER D- = LEFT OF THE RESISTER"
Changed lines of the file:
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@@
 		)
 	)
-	(gr_text "GIPO13"
+	(gr_text "GPIO13"
 		(at 132 113.5 0)
 		(layer "F.SilkS")
@@
 		)
 	)
-	(gr_text "GIPO10"
+	(gr_text "GPIO10"
 		(at 99 112 0)
 		(layer "F.SilkS")
@@
 		)
 	)
-	(gr_text "GIPO1"
+	(gr_text "GPIO1"
 		(at 104 68 0)
 		(layer "F.SilkS")
@@
 		)
 	)
-	(gr_text "GIPO15"
+	(gr_text "GPIO15"
 		(at 120 113.5 0)
 		(layer "F.SilkS")
@@
 		)
 	)
-	(gr_text "GIPO0"
+	(gr_text "GPIO0"
 		(at 110 68 0)
 		(layer "F.SilkS")
@@
 		)
 	)
-	(gr_text "GIPO3"
+	(gr_text "GPIO3"
 		(at 93 68 0)
 		(layer "F.SilkS")
@@
 		)
 	)
-	(gr_text "GIPO11"
+	(gr_text "GPIO11"
 		(at 93 112 0)
 		(layer "F.SilkS")
@@
 		)
 	)
-	(gr_text "GIPO6"
+	(gr_text "GPIO6"
 		(at 104 86 0)
 		(layer "F.SilkS")
@@
 		)
 	)
-	(gr_text "GIPO8\n"
+	(gr_text "GPIO8\n"
 		(at 110 112 0)
 		(layer "F.SilkS")
@@
 		)
 	)
-	(gr_text "GIPO9"
+	(gr_text "GPIO9"
 		(at 105 112 0)
 		(layer "F.SilkS")
@@
 		)
 	)
-	(gr_text "GIPO5\n"
+	(gr_text "GPIO5\n"
 		(at 98.5 86 0)
 		(layer "F.SilkS")
@@
 		)
 	)
-	(gr_text "GIPO7"
+	(gr_text "GPIO7"
 		(at 109 86 0)
 		(layer "F.SilkS")
@@
 		)
 	)
-	(gr_text "GIPO2"
+	(gr_text "GPIO2"
 		(at 98.5 68 0)
 		(layer "F.SilkS")
@@
 		)
 	)
-	(gr_text "GIPO12"
+	(gr_text "GPIO12"
 		(at 138 113.5 0)
 		(layer "F.SilkS")
@@
 		)
 	)
-	(gr_text "GIPO14"
+	(gr_text "GPIO14"
 		(at 126 113.5 0)
 		(layer "F.SilkS")
@@
 		)
 	)
-	(gr_text "GIPO4"
+	(gr_text "GPIO4"
 		(at 93 86 0)
 		(layer "F.SilkS")
@@
 		)
 	)
-	(gr_text "          REFF FOR BAORD \nD- = DATA THEN LINE OUPUT NUMBER\n1  = A NUMBER BY ITS LEFT NEXT TO THE \nPICO LABLES THE GPIO NUMBER OF THAT PIN\n                TEST POINTS\nGPIO = RIGHT OF RESISTER \nD-   = LEFT OF THE RESISTER\n"
+	(gr_text "          REF FOR BOARD \nD- = DATA THEN LINE OUPUT NUMBER\n1  = A NUMBER BY ITS LEFT NEXT TO THE \nPICO LABLES THE GPIO NUMBER OF THAT PIN\n                TEST POINTS\nGPIO = RIGHT OF RESISTOR \nD-   = LEFT OF THE RESISTOR\n"
 		(at 146 126 0)
 		(layer "F.SilkS")
@@
 		)
 	)
-	(gr_text "PCB DESIGNED BY SAMSON B \nLEEDS HACKSPACE CUBE CONTROLL BAORD\nCAN BE FOUND ON GITHUB AT \nwww.github.com/bozzer91\nIF NOT ON LEEDS HACKSPACE GITHUB \nLICENCE: OPEN SOURCE"
+	(gr_text "PCB DESIGNED BY SAMSON B \nLEEDS HACKSPACE CUBE CONTROL BOARD\nCAN BE FOUND ON GITHUB AT \nwww.github.com/bozzer91\nIF NOT ON LEEDS HACKSPACE GITHUB \nLICENCE: OPEN SOURCE"
 		(at 166.5 127.5 0)
 		(layer "B.SilkS")

Commit message: fixed more spelling
Parts:
- renumbered 3M to M3
Changed lines of the file:
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@@
 		(descr "Mounting Hole 3.2mm, M3, generated by kicad-footprint-generator mountinghole.py")
 		(tags "mountinghole M3 ISO7380")
-		(property "Reference" "3M"
+		(property "Reference" "M3"
 			(at 0 -3.8 0)
 			(layer "F.SilkS")
